File: ServoController/ServoController.kicad_sch (KiCad schematic)
At the start: 1 part, among them U1 AS5600

Commit message: main parts
Parts:
- added U2: ATmega328P-P, Package_DIP:DIP-28_W7.62mm, symbol MCU_Microchip_ATmega:ATmega328P-P
- added U3: DRV8231DDAR, DRV8231DDAR:IC_DRV8231DDAR, symbol DRV8231DDAR:DRV8231DDAR
Connections:
- new net: U2.22 (GND), U2.8 (GND)
Other:
- moved on the sheet: U1
